File: versions/v0.9.2/hardware/KiCad_files/PCB layout/prototype.kicad_pcb (KiCad board)
At the start: 2 copper layers, 50 x 42.2 mm, 31 parts, among them P1 CONN_01X02, P2 CONN_01X12, P3 CONN_01X10, P4 CONN_01X01, P5 CONN_01X01, U1 EL3H7, U2 FDC1004custom

Commit message: Modernize v0.9.2 KiCad files for KiCad 9
Parts:
- P1: footprint Downey:special_Header_Straight_1x02_Pitch2.52mm -> Pin_Headers:Pin_Header_Straight_1x02_Pitch2.00mm
- R1, R2: moved to F.Cu
- moved U1 4.76 mm to (166.1, 91.9), turned to -90 degrees
- moved P1 4.46 mm to (160.0, 91.9), turned to -90 degrees
- moved GND1 3.69 mm to (166.1, 87.6)
- moved R1 2.50 mm to (160.0, 87.9), turned to 180 degrees
- moved R2 1.31 mm to (167.8, 95.2)
Routing:
- net Net-(R1-Pad1): track 13.9 -> 4.05 mm, vias 1 -> 0
- net GNDA: track 221.9 -> 229.4 mm, vias 11 -> 12
- net +5V: track 56.1 -> 50.9 mm
- net trigger: track 52.1 -> 55.2 mm, vias 0 -> 1
- net Net-(P1-Pad1): track 6.13 -> 3.76 mm
Other:
- board text added: "IESS Single Board DAQ V0.1d January 2017 Austin R.J. Downey"
- board text added: "IESS v0.1d"
- board text removed: "CDC"
- board text removed: "GND"
- board text removed: "SEC DAQ V0.2b February 2017 Austin R.J. Downey"
- board text removed: "SEC DAQ v0.2b Austin R.J. Downey"
- board text removed: "filter"
